Commit message: color is added

File: mira_description/urdf/mira_simple.urdf (robot description, URDF)
Before this commit: robot mira, 2 links, 1 joints
Links:
- link base_link: geometry visual cylinder length=0.2 radius=0.06
- link roll_M1_link: geometry visual cylinder length=0.2 radius=0.06
Joints:
- joint roll_joint: origin xyz=0.0023 0 -0.0005 rpy=0 0 0 -> xyz=0.0 0.0 0.1 rpy=0 0 0
